File: hardware/erun/erun.sch (KiCad schematic (older format))
At the start: 7 parts

Commit message: hardware
Parts:
- added J? (x2): DB15_Female_MountingHoles, symbol Connector:DB15_Female_MountingHoles
- added J?: Conn_Coaxial, symbol Connector:Conn_Coaxial
- added J?: DB9_Male_MountingHoles, symbol Connector:DB9_Male_MountingHoles
- added U?: MCP3301, symbol Analog_ADC:MCP3301
- added U?: LF47_TO252, Package_TO_SOT_SMD:TO-252-2, symbol Regulator_Linear:LF47_TO252
- added U?: MC3487DX, Package_SO:SOIC-16_3.9x9.9mm_P1.27mm, symbol Interface_LineDriver:MC3487DX
- U?: symbol teensy:Teensy4.0 -> erun-rescue:Teensy4.0-teensy
Connections:
- net labels added: +3.3V, +5V, ADC_IN5V, ADC_INGND, ADC_REF, CLK_HV, CS_HV, DOUT_HV, GND, HV_REF, LLC_OE, LV_REF, S1_A0, S1_A0_HV, S1_A0_HV+, S1_A0_HV-, S1_A1, S1_A1_HV, S1_A1_HV+, S1_A1_HV-, S1_AS_HV+, S1_AS_HV-, S1_B, S1_B_HV, S1_B_HV+, S1_B_HV-, TRIGOUT1_HV+, TRIGOUT1_HV-
- wire segments 0 -> 69
Other:
- note added: "ADC"
- note added: "CONNECTORS\n"
- note added: "DIFFERENTIAL CONVERTER\n"
- moved on the sheet: U?, U?A, U?B, U?C, U?D

Commit message: Updated schematic
Connections:
- net S1_A0 is gone; now on net S1_A0_LV: U?.10 (A8)
- net S1_A1 is gone; now on net S1_B_LV: U?.8 (A6)
- net S1_B is gone; now on net S1_A1_LV: U?.9 (A7)
- net +5V: now also J?.4
- net CLK_HV: no longer U?.3 (A3)
- net CS_HV: no longer U?.1 (A1)
- net DOUT_HV: no longer U?.2 (A2)
- net GND: now also J?.2
- net S1_A0_HV: now also U?.11 (B8); no longer U?.13 (B6)
- net S1_A0_HV+: now also J?.14 (P14)
- net S1_A0_HV-: now also J?.7
- net S1_A1_HV: now also U?.12 (B7); no longer U?.11 (B8)
- net S1_A1_HV+: now also J?.1
- net S1_A1_HV-: now also J?.9 (P9)
- net S1_B_HV: now also U?.13 (B6); no longer U?.12 (B7)
- net S1_B_HV+: now also J?.3
- net S1_B_HV-: now also J?.11 (P111)
- net CS_LV: now reaches U?.12 (10_CS_MQSR)
- net CS_LV: now also U?.3 (A3)
- net DOUT_LV: now reaches U?.14 (12_MISO_MQSL)
- net DOUT_LV: now also U?.2 (A2)
- net CLK_LV: now reaches U?.20 (13_SCK_CRX1_LED)
- net CLK_LV: now also U?.1 (A1)
- net S1_A0_LV: now reaches U?.3 (1_TX1_CTX2_MISO1)
- net S1_A1_LV: now reaches U?.4 (2_OUT2)
- net S1_B_LV: now reaches U?.5 (3_LRCLK2)
- net S1_AS_LV: now reaches U?.6 (4_BCLK2)
- net S1_AS_LV: now also U?.7 (A5)
- net S1_AS_HV: now reaches U?.14 (B5)
- net S1_AS_HV: now also J?.13 (P13)
Other:
- note added: "VOLTAGE-LEVEL SHIFTER"
- moved on the sheet: U?A, U?B, U?C, U?D
