File: hardware/erun/erun.sch (KiCad schematic (older format))
At the start: 10 parts, among them J1 Conn_Coaxial, J2 HEIDENHAIN_MT25_TTL, J3 TRIGGER_TTL, U1 LF47_TO252, U2 MCP3301, U3 MC3486N, U4 MC3486N, U5 TXB0108DQSR, U6 TXB0108DQSR, U7 Teensy4.0

Commit message: Updated schematics and PCB design
Parts:
- removed U3, U4: MC3486N, Package_DIP:DIP-14_W7.62mm, symbol Interface_LineDriver:MC3486N
- added U1, U3: MC3486N, MC3486N:DIP794W45P254L1969H508Q16, symbol MC3486N:MC3486N
- J1: renamed from J2; footprint Connector_Dsub:DSUB-44-HD_Female_Vertical_P2.29x1.98mm_MountingHoles -> Connector_Dsub:DSUB-15_Female_Horizontal_P2.77x2.84mm_EdgePinOffset7.70mm_Housed_MountingHolesOffset9.12mm
- J2: renamed from J3; footprint Connector_Dsub:DSUB-44-HD_Female_Vertical_P2.29x1.98mm_MountingHoles -> Connector_Dsub:DSUB-15_Female_Horizontal_P2.77x2.84mm_EdgePinOffset7.70mm_Housed_MountingHolesOffset9.12mm
- U2: renamed from U6; footprint Package_SON:USON-20_2x4mm_P0.4mm -> TXB0108DQSR:SON40P400X200X55-20N
- U6: renamed from U5; footprint Package_SON:USON-20_2x4mm_P0.4mm -> TXB0108DQSR:SON40P400X200X55-20N
- renumbered J1 to J3, U7 to U4, U1 to U5, U2 to U7
Connections:
- net +5V: now also U1.12 (3,4EN), U1.16 (VCC), U1.4 (1,2EN), U3.12 (3,4EN), U3.16 (VCC), U3.4 (1,2EN)
- net ADC_IN5V: now also J3.1 (In); no longer J3.2 (Ext)
- net ADC_INGND: now also J3.2 (Ext); no longer J3.1 (In)
- net GND: now also U1.8 (GND), U3.8 (GND)
- net S1_A0_HV: now also U1.3 (1Y)
- net S1_A0_HV+: now also U1.2 (1A)
- net S1_A0_HV-: now also U1.1 (1B)
- net S1_A1_HV: now also U1.5 (2Y)
- net S1_A1_HV+: now also U1.6 (2A)
- net S1_A1_HV-: now also U1.7 (2B)
- net S1_A2_HV: now also U1.11 (3Y)
- net S1_A2_HV+: now also U1.10 (3A)
- net S1_A2_HV-: now also U1.9 (3B)
- net S2_A0_HV: now also U3.3 (1Y)
- net S2_A0_HV+: now also U3.2 (1A)
- net S2_A0_HV-: now also U3.1 (1B)
- net S2_A1_HV: now also U3.5 (2Y)
- net S2_A1_HV+: now also U3.6 (2A)
- net S2_A1_HV-: now also U3.7 (2B)
- net S2_A2_HV: now also U3.11 (3Y)
- net S2_A2_HV+: now also U3.10 (3A)
- net S2_A2_HV-: now also U3.9 (3B)
Other:
- moved on the sheet: J3, U2, U4, U5, U6, U7

Commit message: Updated schema
Connections:
- net LLC_OE is gone; now on net +5V: U6.6 (OE)
- net +5V: now also U2.6 (OE)
Changed lines of the file:
@@
 	7650 10850 8050 10850
 Text Label 8050 10950 0    50   ~ 0
-LLC_OE
+HV_REF
 Wire Wire Line
 	8050 10950 7650 10950
@@
 Text Label 1850 10750 0    50   ~ 0
 ADC_IN5V
+Text Label 8800 5800 0    50   ~ 0
+HV_REF
+Wire Wire Line
+	8800 5800 8450 5800
 $EndSCHEMATC

Commit message: erun updates
Parts:
- removed U5: LF47_TO252, Package_TO_SOT_SMD:TO-252-2, symbol Regulator_Linear:LF47_TO252
- added C1, C2, C3, C4: C, Capacitor_SMD:C_0603_1608Metric, symbol Device:C
- added U5: TPS793475-EP, Package_TO_SOT_SMD:SOT-23-5, symbol Regulator_Linear:TPS793475-EP
- J3: footprint Connector_Coaxial:BNC_Amphenol_031-6575_Horizontal -> Connector_Coaxial:SMA_Amphenol_132134-14_Vertical
- U1, U3: footprint MC3486N:DIP794W45P254L1969H508Q16 -> Package_SO:SOIC-16_4.55x10.3mm_P1.27mm
- U2, U6: footprint TXB0108DQSR:SON40P400X200X55-20N -> Package_SO:TSSOP-20_4.4x6.5mm_P0.65mm
- U7: footprint MCP3301:DIP254P762X432-8 -> Package_SO:MSOP-8_3x3mm_P0.65mm
Connections:
- net +3V3: now also U2.6 (OE), U4.31 (3V3), U6.6 (OE); no longer U4.34 (VUSB)
- net +5V: now also U4.34 (VUSB), C1.1, C4.1, U5.1 (IN); no longer U2.6 (OE), U4.35 (24_A10_TX6_SCL2), U6.6 (OE)
- net ADC_REF: now also C3.1, U5.5 (OUT)
- net GND: now also J1.0 (PAD), J2.0 (PAD), U4.1 (GND), U4.32 (GND), C1.2, C2.2, C3.2, C4.2, U5.2 (GND), U5.3 (EN)
- new net: C2.1, U5.4 (BP)
- no-connect marks 0 -> 62
Other:
- moved on the sheet: U7
