File: hardware/erun/_autosave-erun.sch (KiCad schematic (older format))
At the start: 10 parts, among them J1 Conn_Coaxial, J2 HEIDENHAIN_MT25_TTL, J3 TRIGGER_TTL, U1 LF47_TO252, U2 MCP3301, U3 MC3486N, U4 MC3486N, U5 TXB0108DQSR, U6 TXB0108DQSR, U7 Teensy4.0

Commit message: Updated schematics
Parts:
- renumbered J2 to J1, J3 to J2, J1 to J3, U3 to U1, U6 to U2, U4 to U3, U7 to U4, U1 to U5, U5 to U6, U2 to U7
Changed lines of the file:
@@
 $EndDescr
 $Comp
-L erun-rescue:Teensy4.0-teensy U7
+L erun-rescue:Teensy4.0-teensy U4
 U 1 1 618C47F0
 P 10850 8950
-F 0 "U7" H 10850 10565 50  0000 C CNN
+F 0 "U4" H 10850 10565 50  0000 C CNN
 F 1 "Teensy4.0" H 10850 10474 50  0000 C CNN
 F 2 "teensy:Teensy40" H 10450 9150 50  0001 C CNN
@@
 S1_A0_HV-
 $Comp
-L Interface_LineDriver:MC3486N U3
+L Interface_LineDriver:MC3486N U1
 U 1 1 618BF9C9
 P 4600 1350
-F 0 "U3" H 5144 1396 50  0000 L CNN
+F 0 "U1" H 5144 1396 50  0000 L CNN
 F 1 "MC3486N" H 5144 1305 50  0000 L CNN
 F 2 "Package_DIP:DIP-14_W7.62mm" H 4600 950 50  0001 C CNN
@@
 $EndComp
 $Comp
-L power:+3.3V #PWR017
+L power:+3.3V #PWR014
 U 1 1 6198B2D9
 P 12200 9800
-F 0 "#PWR017" H 12200 9650 50  0001 C CNN
+F 0 "#PWR014" H 12200 9650 50  0001 C CNN
 F 1 "+3.3V" H 12215 9973 50  0000 C CNN
 F 2 "" H 12200 9800 50  0001 C CNN
@@
 LV_REF
 $Comp
-L power:+5V #PWR016
+L power:+5V #PWR012
 U 1 1 6198BB4C
 P 12200 9500
-F 0 "#PWR016" H 12200 9350 50  0001 C CNN
+F 0 "#PWR012" H 12200 9350 50  0001 C CNN
 F 1 "+5V" H 12215 9673 50  0000 C CNN
 F 2 "" H 12200 9500 50  0001 C CNN
@@
 HV_REF
 $Comp
-L power:GND #PWR015
+L power:GND #PWR011
 U 1 1 619B8330
 P 8700 9400
-F 0 "#PWR015" H 8700 9150 50  0001 C CNN
+F 0 "#PWR011" H 8700 9150 50  0001 C CNN
 F 1 "GND" H 8705 9227 50  0000 C CNN
 F 2 "" H 8700 9400 50  0001 C CNN
@@
 	4600 1650 4900 1650
 $Comp
-L power:GND #PWR05
+L power:GND #PWR02
 U 1 1 619ED40F
 P 4300 2700
-F 0 "#PWR05" H 4300 2450 50  0001 C CNN
+F 0 "#PWR02" H 4300 2450 50  0001 C CNN
 F 1 "GND" H 4305 2527 50  0000 C CNN
 F 2 "" H 4300 2700 50  0001 C CNN
@@
 $EndComp
 $Comp
-L power:GND #PWR03
+L power:GND #PWR01
 U 1 1 619F196B
 P 4200 1650
-F 0 "#PWR03" H 4200 1400 50  0001 C CNN
+F 0 "#PWR01" H 4200 1400 50  0001 C CNN
 F 1 "GND" H 4205 1477 50  0000 C CNN
 F 2 "" H 4200 1650 50  0001 C CNN
@@
 	2350 2150 2100 2150
 $Comp
-L power:GND #PWR01
+L power:GND #PWR03
 U 1 1 619E3C39
 P 2850 3150
-F 0 "#PWR01" H 2850 2900 50  0001 C CNN
+F 0 "#PWR03" H 2850 2900 50  0001 C CNN
 F 1 "GND" H 2855 2977 50  0000 C CNN
 F 2 "" H 2850 3150 50  0001 C CNN
@@
 	2100 2850 2200 2850
 $Comp
-L Connector:DB15_Female_MountingHoles J2
+L Connector:DB15_Female_MountingHoles J1
 U 1 1 61970C5D
 P 1800 2350
-F 0 "J2" H 1955 2352 50  0000 L CNN
+F 0 "J1" H 1955 2352 50  0000 L CNN
 F 1 "HEIDENHAIN_MT25_TTL" H 1955 2261 50  0000 L CNN
 F 2 "Connector_Dsub:DSUB-44-HD_Female_Vertical_P2.29x1.98mm_MountingHoles" H 1800 2350 50  0001 C CNN
@@
 S1_AS_LV
 $Comp
-L Logic_LevelTranslator:TXB0108DQSR U6
+L Logic_LevelTranslator:TXB0108DQSR U2
 U 1 1 618C6CB9
 P 7850 5400
-F 0 "U6" H 7850 4611 50  0000 C CNN
+F 0 "U2" H 7850 4611 50  0000 C CNN
 F 1 "TXB0108DQSR" H 7850 4520 50  0000 C CNN
 F 2 "Package_SON:USON-20_2x4mm_P0.4mm" H 7850 4650 50  0001 C CNN
@@
 	7850 4700 7850 4400
 $Comp
-L power:GND #PWR014
+L power:GND #PWR05
 U 1 1 61998562
 P 8550 4550
-F 0 "#PWR014" H 8550 4300 50  0001 C CNN
+F 0 "#PWR05" H 8550 4300 50  0001 C CNN
 F 1 "GND" H 8555 4377 50  0000 C CNN
 F 2 "" H 8550 4550 50  0001 C CNN
@@
 HV_REF
 $Comp
-L Connector:DB15_Female_MountingHoles J3
+L Connector:DB15_Female_MountingHoles J2
 U 1 1 61E7C7DB
 P 1800 7000
-F 0 "J3" H 1955 7002 50  0000 L CNN
+F 0 "J2" H 1955 7002 50  0000 L CNN
 F 1 "TRIGGER_TTL" H 1955 6911 50  0000 L CNN
 F 2 "Connector_Dsub:DSUB-44-HD_Female_Vertical_P2.29x1.98mm_MountingHoles" H 1800 7000 50  0001 C CNN
@@
 	2100 7500 2200 7500
 $Comp
-L power:GND #PWR02
+L power:GND #PWR09
 U 1 1 61E7C7D4
 P 2850 7800
-F 0 "#PWR02" H 2850 7550 50  0001 C CNN
+F 0 "#PWR09" H 2850 7550 50  0001 C CNN
 F 1 "GND" H 2855 7627 50  0000 C CNN
 F 2 "" H 2850 7800 50  0001 C CNN
@@
 S1_A2_HV-
 $Comp
-L Interface_LineDriver:MC3486N U3
+L Interface_LineDriver:MC3486N U1
 U 2 1 618BDA93
 P 4600 2400
-F 0 "U3" H 5144 2446 50  0000 L CNN
+F 0 "U1" H 5144 2446 50  0000 L CNN
 F 1 "MC3486N" H 5144 2355 50  0000 L CNN
 F 2 "Package_DIP:DIP-14_W7.62mm" H 4600 2000 50  0001 C CNN
@@
 	4600 3800 4900 3800
 $Comp
-L Interface_LineDriver:MC3486N U3
+L Interface_LineDriver:MC3486N U1
 U 3 1 618C0C51
 P 4600 3500
-F 0 "U3" H 5144 3546 50  0000 L CNN
+F 0 "U1" H 5144 3546 50  0000 L CNN
 F 1 "MC3486N" H 5144 3455 50  0000 L CNN
 F 2 "Package_DIP:DIP-14_W7.62mm" H 4600 3100 50  0001 C CNN
@@
 	4300 3800 4500 3800
 $Comp
-L power:GND #PWR06
+L power:GND #PWR04
 U 1 1 619F2EB7
 P 4300 3800
-F 0 "#PWR06" H 4300 3550 50  0001 C CNN
+F 0 "#PWR04" H 4300 3550 50  0001 C CNN
 F 1 "GND" H 4305 3627 50  0000 C CNN
 F 2 "" H 4300 3800 50  0001 C CNN
@@
 S2_A0_HV-
 $Comp
-L Interface_LineDriver:MC3486N U4
+L Interface_LineDriver:MC3486N U3
 U 1 1 625D4659
 P 4600 6050
-F 0 "U4" H 5144 6096 50  0000 L CNN
+F 0 "U3" H 5144 6096 50  0000 L CNN
 F 1 "MC3486N" H 5144 6005 50  0000 L CNN
 F 2 "Package_DIP:DIP-14_W7.62mm" H 4600 5650 50  0001 C CNN
@@
 $EndComp
 $Comp
-L power:GND #PWR04
+L power:GND #PWR07
 U 1 1 625D4667
 P 4200 6350
-F 0 "#PWR04" H 4200 6100 50  0001 C CNN
+F 0 "#PWR07" H 4200 6100 50  0001 C CNN
 F 1 "GND" H 4205 6177 50  0000 C CNN
 F 2 "" H 4200 6350 50  0001 C CNN
@@
 S2_A2_HV-
 $Comp
-L Interface_LineDriver:MC3486N U4
+L Interface_LineDriver:MC3486N U3
 U 2 1 625D4670
 P 4600 7100
-F 0 "U4" H 5144 7146 50  0000 L CNN
+F 0 "U3" H 5144 7146 50  0000 L CNN
 F 1 "MC3486N" H 5144 7055 50  0000 L CNN
 F 2 "Package_DIP:DIP-14_W7.62mm" H 4600 6700 50  0001 C CNN
@@
 	4600 8500 4900 8500
 $Comp
-L Interface_LineDriver:MC3486N U4
+L Interface_LineDriver:MC3486N U3
 U 3 1 625D4683
 P 4600 8200
-F 0 "U4" H 5144 8246 50  0000 L CNN
+F 0 "U3" H 5144 8246 50  0000 L CNN
 F 1 "MC3486N" H 5144 8155 50  0000 L CNN
 F 2 "Package_DIP:DIP-14_W7.62mm" H 4600 7800 50  0001 C CNN
@@
 	4300 8500 4500 8500
 $Comp
-L power:GND #PWR09
+L power:GND #PWR010
 U 1 1 625D4691
 P 4300 8500
-F 0 "#PWR09" H 4300 8250 50  0001 C CNN
+F 0 "#PWR010" H 4300 8250 50  0001 C CNN
 F 1 "GND" H 4305 8327 50  0000 C CNN
 F 2 "" H 4300 8500 50  0001 C CNN
@@
 	1450 11400 1450 11600
 $Comp
-L Connector:Conn_Coaxial J1
+L Connector:Conn_Coaxial J3
 U 1 1 619E4137
 P 1450 11800
-F 0 "J1" H 1550 11775 50  0000 L CNN
+F 0 "J3" H 1550 11775 50  0000 L CNN
 F 1 "Conn_Coaxial" H 1550 11684 50  0000 L CNN
 F 2 "Connector_Coaxial:BNC_Amphenol_031-6575_Horizontal" H 1450 11800 50  0001 C CNN
@@
 HV_REF
 $Comp
-L Analog_ADC:MCP3301 U2
+L Analog_ADC:MCP3301 U7
 U 1 1 61966194
 P 4150 11800
-F 0 "U2" H 4100 11219 50  0000 C CNN
+F 0 "U7" H 4100 11219 50  0000 C CNN
 F 1 "MCP3301" H 4100 11310 50  0000 C CNN
 F 2 "MCP3301:DIP254P762X432-8" H 4950 11700 50  0001 C CNN
@@
 	4150 10650 4150 10500
 $Comp
-L Regulator_Linear:LF47_TO252 U1
+L Regulator_Linear:LF47_TO252 U5
 U 1 1 619A3A45
 P 4150 10950
-F 0 "U1" H 4150 11192 50  0000 C CNN
+F 0 "U5" H 4150 11192 50  0000 C CNN
 F 1 "LF47_TO252" H 4150 11101 50  0000 C CNN
 F 2 "Package_TO_SOT_SMD:TO-252-2" H 4150 11175 50  0001 C CIN
@@
 	4050 11300 4050 11400
 $Comp
-L power:GND #PWR011
+L power:GND #PWR017
 U 1 1 6198A32B
 P 4050 12400
-F 0 "#PWR011" H 4050 12150 50  0001 C CNN
+F 0 "#PWR017" H 4050 12150 50  0001 C CNN
 F 1 "GND" H 4055 12227 50  0000 C CNN
 F 2 "" H 4050 12400 50  0001 C CNN
@@
 	3200 11900 3550 11900
 $Comp
-L power:GND #PWR012
+L power:GND #PWR015
 U 1 1 619A1D4F
 P 4350 10500
-F 0 "#PWR012" H 4350 10250 50  0001 C CNN
+F 0 "#PWR015" H 4350 10250 50  0001 C CNN
 F 1 "GND" H 4355 10327 50  0000 C CNN
 F 2 "" H 4350 10500 50  0001 C CNN
@@
 	7350 12550 7350 12300
 $Comp
-L power:GND #PWR013
+L power:GND #PWR016
 U 1 1 61E5DBC3
 P 7950 10750
-F 0 "#PWR013" H 7950 10500 50  0001 C CNN
+F 0 "#PWR016" H 7950 10500 50  0001 C CNN
 F 1 "GND" H 7955 10577 50  0000 C CNN
 F 2 "" H 7950 10750 50  0001 C CNN
@@
 	7950 10600 7950 10750
 $Comp
-L Logic_LevelTranslator:TXB0108DQSR U5
+L Logic_LevelTranslator:TXB0108DQSR U6
 U 1 1 61E3A167
 P 7250 11600
-F 0 "U5" H 7250 10719 50  0000 C CNN
+F 0 "U6" H 7250 10719 50  0000 C CNN
 F 1 "TXB0108DQSR" H 7250 10810 50  0000 C CNN
 F 2 "Package_SON:USON-20_2x4mm_P0.4mm" H 7250 10850 50  0001 C CNN
@@
 	4600 4750 4900 4750
 $Comp
-L Interface_LineDriver:MC3486N U3
+L Interface_LineDriver:MC3486N U1
 U 4 1 62659DD4
 P 4600 4450
-F 0 "U3" H 5144 4496 50  0000 L CNN
+F 0 "U1" H 5144 4496 50  0000 L CNN
 F 1 "MC3486N" H 5144 4405 50  0000 L CNN
 F 2 "Package_DIP:DIP-14_W7.62mm" H 4600 4050 50  0001 C CNN
@@
 	4300 4750 4500 4750
 $Comp
-L power:GND #PWR07
+L power:GND #PWR06
 U 1 1 62659DE2
 P 4300 4750
-F 0 "#PWR07" H 4300 4500 50  0001 C CNN
+F 0 "#PWR06" H 4300 4500 50  0001 C CNN
 F 1 "GND" H 4305 4577 50  0000 C CNN
 F 2 "" H 4300 4750 50  0001 C CNN
@@
 	4600 9550 4900 9550
 $Comp
-L Interface_LineDriver:MC3486N U4
+L Interface_LineDriver:MC3486N U3
 U 4 1 626CC157
 P 4600 9250
-F 0 "U4" H 5144 9296 50  0000 L CNN
+F 0 "U3" H 5144 9296 50  0000 L CNN
 F 1 "MC3486N" H 5144 9205 50  0000 L CNN
 F 2 "Package_DIP:DIP-14_W7.62mm" H 4600 8850 50  0001 C CNN
@@
 	4300 9550 4500 9550
 $Comp
-L power:GND #PWR010
+L power:GND #PWR013
 U 1 1 626CC165
 P 4300 9550
-F 0 "#PWR010" H 4300 9300 50  0001 C CNN
+F 0 "#PWR013" H 4300 9300 50  0001 C CNN
 F 1 "GND" H 4305 9377 50  0000 C CNN
 F 2 "" H 4300 9550 50  0001 C CNN
